Commit message: added google cartographer video on 2d mapping

File: models/urdf/simplebot.xacro (robot description, xacro)
@@ -85,4 +85,5 @@
   </collision>
 </link>
+<link name="camera"></link>
 <link name="lidar_1">
   <inertial>
@@ -122,4 +123,9 @@
   <child link="caster_wheel_1"/>
 </joint>
+<joint name="camera_joint" type="fixed">
+  <origin xyz="0.0 0.0 0.08" rpy="0 0 0"/>
+  <parent link="base_link"/>
+  <child link="camera"/>
+</joint>
 <joint name="lidar_joint" type="fixed">
   <origin xyz="0.0 0.0 0.0675" rpy="0 0 0"/>
